Commit message: modify can_communication

File: base_description/urdf/xacro/gazebo/mbot_with_laser_gazebo.xacro (robot description, xacro)
@@ -4,11 +4,16 @@
     <xacro:include filename="$(find base_description)/urdf/xacro/sensors/lidar_gazebo.xacro" />
     <xacro:include filename="$(find base_description)/urdf/xacro/sensors/imu_gazebo.xacro" />
+    <!--xacro:include filename="$(find base_description)/urdf/xacro/actuator/aubo_i10.xacro" /-->
     <xacro:property name="lidar_offset_x" value="0.25" />
     <xacro:property name="lidar_offset_y" value="0" />
-    <xacro:property name="lidar_offset_z" value="0.125" />
+    <xacro:property name="lidar_offset_z" value="0.1" />
     <xacro:property name="imu_offset_x" value="0" />
     <xacro:property name="imu_offset_y" value="0" />
     <xacro:property name="imu_offset_z" value="0.125" />
+    <!--xacro:property name="pedestal_offset_x" value="0" />
+    <xacro:property name="pedestal_offset_y" value="0" />
+    <xacro:property name="pedestal_offset_z" value="0.125"/-->
     <mbot_base/>
+    <aubo_i10/>
     <!-- lidar -->
     <joint name="lidar_joint" type="fixed">
@@ -27,4 +32,12 @@
     </joint>
     <xacro:imu prefix="imu"/>
+    <!--aubo_i10 -->
+    <!--joint name="pedestal_joint" type="fixed">
+        <origin xyz="${pedestal_offset_x}
+        ${pedestal_offset_y} ${pedestal_offset_z}" rpy="0 0 0" />
+        <parent link="lift2_link"/>
+        <child link="pedestal_link"/>
+    </joint-->
     <mbot_base_gazebo/>
+    <aubo_i10_gazebo/>
 </robot>

File: base_description/urdf/xacro/mbot_base.xacro (robot description, xacro)
@@ -213,5 +213,5 @@
             </collision>
             <inertial>
-                <mass value="60"/>
+                <mass value="120"/>
                 <inertia ixx="1.0" ixy="0.0" ixz="0.0" iyy="1.0" iyz="0.0" izz="1.0"/>
             </inertial>

File: base_description/urdf/xacro/sensors/lidar_gazebo.xacro (robot description, xacro)
@@ -44,5 +44,5 @@
                     <range>
                       <min>0.10</min>
-                      <max>10.0</max>
+                      <max>100</max>
                       <resolution>0.01</resolution>
                     </range>
